Commit message: update urdf

File: robots/adam_lite/urdf/adam_lite.urdf (robot description, URDF)
Before this commit: robot adam_lite, 28 links, 27 joints
Joints:
- joint hipPitch_Left: limit lower=-2.09 upper=2.09 effort=230.0 velocity=15.0 -> lower=-2.09 upper=2.09 effort=300.0 velocity=15.0
- joint hipPitch_Right: limit lower=-2.09 upper=2.09 effort=230.0 velocity=15.0 -> lower=-2.09 upper=2.09 effort=300.0 velocity=15.0
- joint kneePitch_Left: limit lower=-0.09 upper=2.4 effort=230.0 velocity=15.0 -> lower=-0.09 upper=2.4 effort=300.0 velocity=15.0
- joint kneePitch_Right: limit lower=-0.09 upper=2.4 effort=230.0 velocity=15.0 -> lower=-0.09 upper=2.4 effort=300.0 velocity=15.0

File: robots/adam_lite/urdf/adam_lite_wrist.urdf (robot description, URDF)
Before this commit: robot adam_lite, 28 links, 27 joints
Joints:
- joint hipPitch_Left: limit lower=-2.09 upper=2.09 effort=230.0 velocity=15.0 -> lower=-2.09 upper=2.09 effort=300.0 velocity=15.0
- joint hipPitch_Right: limit lower=-2.09 upper=2.09 effort=230.0 velocity=15.0 -> lower=-2.09 upper=2.09 effort=300.0 velocity=15.0
- joint kneePitch_Left: limit lower=-0.09 upper=2.4 effort=230.0 velocity=15.0 -> lower=-0.09 upper=2.4 effort=300.0 velocity=15.0
- joint kneePitch_Right: limit lower=-0.09 upper=2.4 effort=230.0 velocity=15.0 -> lower=-0.09 upper=2.4 effort=300.0 velocity=15.0

Commit message: add fake wrist joint

File: robots/adam_lite/urdf/adam_lite.urdf (robot description, URDF)
Before this commit: robot adam_lite, 28 links, 27 joints
Links:
- added link wristLeft; visual sphere radius=0.035
- added link wristRight; visual sphere radius=0.035
Joints:
- added joint wrist_Left: type revolute, parent elbowLeft, child wristLeft, origin xyz=-0.0150000000000083 0.0285000000000339 -0.3034000000000177 rpy=0 0 0, axis 0 0 1, limit lower=-3.14 upper=3.14 effort=30.0 velocity=8.0
- added joint wrist_Right: type revolute, parent elbowRight, child wristRight, origin xyz=-0.0149999999999991 -0.0285000000000092 -0.3033999999999902 rpy=0 0 0, axis 0 0 1, limit lower=-3.14 upper=3.14 effort=30.0 velocity=8.0

Commit message: add fixed wrist joint

File: robots/adam_lite/urdf/adam_lite.urdf (robot description, URDF)
Before this commit: robot adam_lite, 30 links, 29 joints
Joints:
- joint wrist_Left: limit lower=-3.14 upper=3.14 effort=30.0 velocity=8.0 -> (none); type revolute -> fixed
- joint wrist_Right: type revolute -> fixed

Commit message: add standard

File: robots/adam_lite/urdf/adam_lite.urdf (robot description, URDF)
Before this commit: robot adam_lite, 30 links, 29 joints
Links:
- removed link footLeftY
- removed link footRightY
- removed link shin_Left
- removed link shin_Right
- removed link shoulderBaseLeft
- removed link shoulderBaseRight
- removed link thigh_Left
- removed link thigh_Right
- removed link toe_left
- removed link toe_right
- removed link wristLeft
- removed link wristRight
- added link anklePitchLeft, mass 0.03100000; visual mesh filename=../meshes/anklePitchLeft.STL
- added link anklePitchRight, mass 0.03100000; visual mesh filename=../meshes/anklePitchRight.STL
- added link shinLeft, mass 2.19866469; collision box size=0.08 0.06 0.3; visual mesh filename=../meshes/shinLeft.STL
- added link shinRight, mass 2.20809154; collision box size=0.08 0.06 0.3; visual mesh filename=../meshes/shinRight.STL
- added link thighLeft, mass 6.64749717; visual mesh filename=../meshes/thighLeft.STL
- added link thighRight, mass 6.64754534; visual mesh filename=../meshes/thighRight.STL
- added link toeLeft, mass 0.47580000; collision box size=0.24 0.1 0.03; visual mesh filename=../meshes/toeLeft.STL
- added link toeRight, mass 0.47580000; collision box size=0.24 0.1 0.03; visual mesh filename=../meshes/toeRight.STL
- link elbowLeft: mass 0.6 -> 0.85400000; geometry visual mesh filename=../meshes/elbowLeft.STL
- link elbowRight: mass 0.6 -> 0.85400000; geometry visual mesh filename=../meshes/elbowRight.STL
- link hipPitchLeft: mass 2.122960 -> 2.15124786
- link hipPitchRight: mass 2.122960 -> 2.15124254
- link hipRollLeft: mass 1.302398 -> 1.29421887
- link hipRollRight: mass 1.302398 -> 1.29422777
- link pelvis: mass 9.240301 -> 10.18730021
- link shoulderPitchLeft: mass 0.222453128267368 -> 0.20310000
- link shoulderPitchRight: mass 0.222453128267368 -> 0.20310000
- link shoulderRollLeft: mass 0.6 -> 0.72480000
- link shoulderRollRight: mass 0.6 -> 0.72480000
- link shoulderYawLeft: mass 0.853573592139701 -> 0.69630000
- link shoulderYawRight: mass 0.853573592139701 -> 0.69630000
- link torso: mass 10.464000 -> 13.28595962
- link waistPitch: mass 0.654478 -> 0.49870000
- link waistRoll: mass 2.50 -> 2.18430742
- link wristYawLeft: mass 0.276361 -> 0.73460000; geometry visual mesh filename=../meshes/wristYawLeft.STL
- link wristYawRight: mass 0.276361 -> 0.73460000; geometry visual mesh filename=../meshes/wristYawRight.STL
Joints:
- removed joint shoulderBase_Left
- removed joint shoulderBase_Right
- removed joint wrist_Left
- removed joint wrist_Right
- joint anklePitch_Left: child footLeftY -> anklePitchLeft; parent shin_Left -> shinLeft
- joint anklePitch_Right: child footRightY -> anklePitchRight; parent shin_Right -> shinRight
- joint ankleRoll_Left: child toe_left -> toeLeft; parent footLeftY -> anklePitchLeft
- joint ankleRoll_Right: child toe_right -> toeRight; parent footRightY -> anklePitchRight
- joint elbow_Left: origin xyz=0 -0.0285 -0.20365 rpy=0 0 0 -> xyz=0 -0.0285 -0.20415 rpy=0 0 0
- joint elbow_Right: origin xyz=0 0.0285 -0.20365 rpy=0 0 0 -> xyz=0 0.0285 -0.20415 rpy=0 0 0
- joint hipPitch_Left: limit lower=-2.09 upper=2.09 effort=300.0 velocity=15.0 -> lower=-2.09 upper=2.09 effort=230.0 velocity=15.0; origin xyz=0 0.096102 -0.027011 rpy=-0.61087 0 0 -> xyz=0 0.096192 -0.033241 rpy=-0.61087 0 0
- joint hipPitch_Right: limit lower=-2.09 upper=2.09 effort=300.0 velocity=15.0 -> lower=-2.09 upper=2.09 effort=230.0 velocity=15.0; origin xyz=0 -0.096102 -0.027011 rpy=0.61087 0 0 -> xyz=0 -0.096192 -0.033241 rpy=0.61087 0 0
- joint hipYaw_Left: child thigh_Left -> thighLeft
- joint hipYaw_Right: child thigh_Right -> thighRight; origin xyz=0.044 0.0 -0.0525 rpy=0 0 0 -> xyz=0.044 0 -0.0525 rpy=0 0 0
- joint kneePitch_Left: child shin_Left -> shinLeft; limit lower=-0.09 upper=2.4 effort=300.0 velocity=15.0 -> lower=-0.09 upper=2.4 effort=230.0 velocity=15.0; parent thigh_Left -> thighLeft
- joint kneePitch_Right: child shin_Right -> shinRight; limit lower=-0.09 upper=2.4 effort=300.0 velocity=15.0 -> lower=-0.09 upper=2.4 effort=230.0 velocity=15.0; parent thigh_Right -> thighRight
- joint shoulderPitch_Left: origin xyz=-0.0020109 0.0717 -0.0011968 rpy=0 0 0 -> xyz=0 0.16011 0.25742 rpy=0.34907 0 0; parent shoulderBaseLeft -> torso
- joint shoulderPitch_Right: origin xyz=-0.0020109 -0.0717 -0.0011968 rpy=0 0 0 -> xyz=0 -0.16011 0.25742 rpy=-0.34907 0 0; parent shoulderBaseRight -> torso
- joint shoulderRoll_Left: origin xyz=0.0335 0.044 0 rpy=-0.34907 0 0 -> xyz=0.0335 0.0435 0 rpy=-0.34907 0 0
- joint shoulderRoll_Right: origin xyz=0.0335 -0.044 0 rpy=0.34907 0 0 -> xyz=0.0335 -0.0435 0 rpy=0.34907 0 0
- joint shoulderYaw_Left: origin xyz=-0.0335 0.034081 -0.059 rpy=0 0 0 -> xyz=-0.0335 0.034 -0.0585 rpy=0 0 0
- joint shoulderYaw_Right: origin xyz=-0.0335 -0.034081 -0.059 rpy=0 0 0 -> xyz=-0.0335 -0.034 -0.0585 rpy=0 0 0
- joint waistRoll: origin xyz=0 0 0.05023 rpy=0 0 0 -> xyz=0 0 0.044 rpy=0 0 0
- joint waistYaw: origin xyz=0 0 0.056115 rpy=0 0 0 -> xyz=0 0.0005 0.053 rpy=0 0 0
- joint wristYaw_Left: limit (none) -> effort=6.4 velocity=4.9218; origin xyz=-0.0150000000000083 0.0285000000000339 -0.0734000000000177 rpy=0 0 0 -> xyz=-0.025 0.0285 -0.0729 rpy=0 0 0
- joint wristYaw_Right: origin xyz=-0.0149999999999991 -0.0285000000000092 -0.0733999999999902 rpy=0 0 0 -> xyz=-0.025 -0.0285 -0.0729 rpy=0 0 0
